Commit message: 1

File: python/FT_sensor/monkey.urdf (robot description, URDF)
Before this commit: robot box, 3 links, 2 joints
Links:
- link sensor_link: geometry collision mesh filename=monkey.stl; visual mesh filename=monkey.stl

File: python/FT_sensor/object.urdf (robot description, URDF)
Before this commit: robot box, 1 links, 0 joints
Links:
- link box_link: geometry collision box size=0.05 0.05 0.05; visual box size=0.05 0.05 0.05
